Commit message: commit

File: snake_robot/snake_description/urdf/sevenJoints.urdf (robot description, URDF)
Before this commit: robot sevenJointsSnake, 9 links, 8 joints
Links:
- added link base_intermediate_x
- added link base_intermediate_y
- link base_link: geometry visual mesh filename=package://snake_robot/snake_description/meshes/servo.stl scale=0.01 0.01 0.01
- link link2: geometry visual mesh filename=package://snake_robot/snake_description/meshes/servo.stl scale=0.01 0.01 0.01
- link link3: geometry visual mesh filename=package://snake_robot/snake_description/meshes/servo.stl scale=0.01 0.01 0.01
- link link4: geometry visual mesh filename=package://snake_robot/snake_description/meshes/servo.stl scale=0.01 0.01 0.01
- link link5: geometry visual mesh filename=package://snake_robot/snake_description/meshes/servo.stl scale=0.01 0.01 0.01
- link link6: geometry visual mesh filename=package://snake_robot/snake_description/meshes/servo.stl scale=0.01 0.01 0.01
- link link7: geometry visual mesh filename=package://snake_robot/snake_description/meshes/servo.stl scale=0.01 0.01 0.01
- link link8: geometry visual mesh filename=package://snake_robot/snake_description/meshes/servo.stl scale=0.01 0.01 0.01
Joints:
- removed joint fixed
- added joint base_prismatic_x: type prismatic, parent world, child base_intermediate_x, origin xyz=0 0 0 rpy=0 0 0, axis 1 0 0, limit lower=-10 upper=10 effort=1000 velocity=1000
- added joint base_prismatic_y: type prismatic, parent base_intermediate_x, child base_intermediate_y, origin xyz=0 0 0 rpy=0 0 0, axis 0 1 0, limit lower=-10 upper=10 effort=1000 velocity=1000
- added joint base_revolute_z: type continuous, parent base_intermediate_y, child base_link, origin xyz=0 0 0 rpy=0 0 0, axis 0 0 1, limit effort=1000 velocity=1000

Commit message: change urdf

File: snake_robot/snake_description/urdf/sevenJoints.urdf (robot description, URDF)
Before this commit: robot sevenJointsSnake, 11 links, 10 joints
Links:
- removed link base_intermediate_x
- removed link base_intermediate_y
- link base_link: geometry visual mesh filename=package://snake_robot/snake_description/meshes/servo.stl scale=0.001 0.001 0.001
- link link2: geometry visual mesh filename=package://snake_robot/snake_description/meshes/servo.stl scale=0.001 0.001 0.001
- link link3: geometry visual mesh filename=package://snake_robot/snake_description/meshes/servo.stl scale=0.001 0.001 0.001
- link link4: geometry visual mesh filename=package://snake_robot/snake_description/meshes/servo.stl scale=0.001 0.001 0.001
- link link5: geometry visual mesh filename=package://snake_robot/snake_description/meshes/servo.stl scale=0.001 0.001 0.001
- link link6: geometry visual mesh filename=package://snake_robot/snake_description/meshes/servo.stl scale=0.001 0.001 0.001
- link link7: geometry visual mesh filename=package://snake_robot/snake_description/meshes/servo.stl scale=0.001 0.001 0.001
- link link8: geometry visual mesh filename=package://snake_robot/snake_description/meshes/servo.stl scale=0.001 0.001 0.001
Joints:
- removed joint base_prismatic_x
- removed joint base_prismatic_y
- removed joint base_revolute_z
- added joint fixed: type fixed, parent world, child base_link
- joint joint2: origin xyz=0. 0. 0.072 rpy=0. 0. 1.57079632679 -> xyz=0. 0.072 0. rpy=0. 0. 0
- joint joint3: origin xyz=0. 0. 0.072 rpy=0. 0. -1.57079632679 -> xyz=0. 0.072 0. rpy=0. 0. 0
- joint joint4: origin xyz=0. 0. 0.072 rpy=0. 0. 1.57079632679 -> xyz=0. 0.072 0. rpy=0. 0. 0
- joint joint5: origin xyz=0. 0. 0.072 rpy=0. 0. -1.57079632679 -> xyz=0. 0.072 0. rpy=0. 0. 0
- joint joint6: origin xyz=0. 0. 0.072 rpy=0. 0. 1.57079632679 -> xyz=0. 0.072 0. rpy=0. 0. 0
- joint joint7: origin xyz=0. 0. 0.072 rpy=0. 0. -1.57079632679 -> xyz=0. 0.072 0. rpy=0. 0. 0

Commit message: changing urdf

File: snake_robot/snake_description/urdf/sevenJoints.urdf (robot description, URDF)
Before this commit: robot sevenJointsSnake, 9 links, 8 joints
Links:
- added link base_intermediate_x
- added link base_intermediate_y
- link base_link: geometry visual mesh filename=package://snake_robot/snake_description/meshes/servo.stl scale=0.01 0.01 0.01
- link link2: geometry visual mesh filename=package://snake_robot/snake_description/meshes/servo.stl scale=0.01 0.01 0.01
- link link3: geometry visual mesh filename=package://snake_robot/snake_description/meshes/servo.stl scale=0.01 0.01 0.01
- link link4: geometry visual mesh filename=package://snake_robot/snake_description/meshes/servo.stl scale=0.01 0.01 0.01
- link link5: geometry visual mesh filename=package://snake_robot/snake_description/meshes/servo.stl scale=0.01 0.01 0.01
- link link6: geometry visual mesh filename=package://snake_robot/snake_description/meshes/servo.stl scale=0.01 0.01 0.01
- link link7: geometry visual mesh filename=package://snake_robot/snake_description/meshes/servo.stl scale=0.01 0.01 0.01
- link link8: geometry visual mesh filename=package://snake_robot/snake_description/meshes/servo.stl scale=0.01 0.01 0.01
Joints:
- removed joint fixed
- added joint base_prismatic_x: type prismatic, parent world, child base_intermediate_x, origin xyz=0 0 0 rpy=0 0 0, axis 1 0 0, limit lower=-10 upper=10 effort=1000 velocity=1000
- added joint base_prismatic_y: type prismatic, parent base_intermediate_x, child base_intermediate_y, origin xyz=0 0 0 rpy=0 0 0, axis 0 1 0, limit lower=-10 upper=10 effort=1000 velocity=1000
- added joint base_revolute_z: type continuous, parent base_intermediate_y, child base_link, origin xyz=0 0 0 rpy=0 0 0, axis 0 0 1, limit effort=1000 velocity=1000
- joint joint2: origin xyz=0. 0.072 0. rpy=0. 0. 0 -> xyz=0. 0.72 0. rpy=0. 0. 0
- joint joint3: origin xyz=0. 0.072 0. rpy=0. 0. 0 -> xyz=0. 0.72 0. rpy=0. 0. 0
- joint joint4: origin xyz=0. 0.072 0. rpy=0. 0. 0 -> xyz=0. 0.72 0. rpy=0. 0. 0
- joint joint5: origin xyz=0. 0.072 0. rpy=0. 0. 0 -> xyz=0. 0.72 0. rpy=0. 0. 0
- joint joint6: origin xyz=0. 0.072 0. rpy=0. 0. 0 -> xyz=0. 0.72 0. rpy=0. 0. 0
- joint joint7: origin xyz=0. 0.072 0. rpy=0. 0. 0 -> xyz=0. 0.72 0. rpy=0. 0. 0

Commit message: moving forward

File: snake_robot/snake_description/urdf/sevenJoints.urdf (robot description, URDF)
Before this commit: robot sevenJointsSnake, 11 links, 10 joints
Links:
- link link2: mass 100 -> 1000
Joints:
- joint joint1: limit lower=-1 upper=1 effort=0.01 velocity=0.5 -> lower=-1 upper=1 effort=1000 velocity=0.5
- joint joint3: limit lower=-1 upper=1 effort=0.01 velocity=0.5 -> lower=-1 upper=1 effort=1000 velocity=0.5
- joint joint4: limit lower=-1 upper=1 effort=0.01 velocity=0.5 -> lower=-1 upper=1 effort=1000 velocity=0.5
- joint joint5: limit lower=-1 upper=1 effort=0.01 velocity=0.5 -> lower=-1 upper=1 effort=1000 velocity=0.5
- joint joint6: limit lower=-1 upper=1 effort=0.01 velocity=0.5 -> lower=-1 upper=1 effort=1000 velocity=0.5
- joint joint7: limit lower=-1 upper=1 effort=0.01 velocity=0.5 -> lower=-1 upper=1 effort=1000 velocity=0.5

Commit message: running but not working code cant solve for djacbian

File: snake_robot/snake_description/urdf/sevenJoints.urdf (robot description, URDF)
Before this commit: robot sevenJointsSnake, 11 links, 10 joints
Links:
- link base_link: mass 1 -> 100
- link link2: mass 1000 -> 100
